File: KiCad/FA-DAC.kicad_pcb (KiCad board)
At the start: 2 copper layers, 80 x 43 mm, 103 parts, among them J100 Conn_02x10_Odd_Even, J101 Conn_01x03_Male, J102 Conn_01x02_Male, J103 Conn_01x02_Male, U200 AD1955, U300 AD797, U301 AD797, U302 AD797, U400 AD797, U401 AD797, U402 AD797

Commit message: Update for release
Parts:
- removed NT1: Net-Tie_2, NetTie:NetTie-2_SMD_Pad0.5mm
- added C1: 4.7u, Capacitor_SMD:C_0402_1005Metric, F.Cu at (-29.8, 15.2)
- added C2: 100n, Capacitor_SMD:C_0402_1005Metric, F.Cu at (-29.8, 14.2)
- added C202: 47u, Capacitor_SMD:C_0805_2012Metric, F.Cu at (-11.8, -6.00)
- added C3: 10n, Capacitor_SMD:C_0402_1005Metric, F.Cu at (-29.8, 7.25)
- added C4: 1u, Capacitor_SMD:C_0402_1005Metric, F.Cu at (-29.8, 6.25)
- added J104: TC2030, Connector:Tag-Connect_TC2030-IDC-NL_2x03_P1.27mm_Vertical, B.Cu at (-20.5, 18.0)
- added Q100: BC856W, Package_TO_SOT_SMD:SOT-323_SC-70, F.Cu at (-21.2, -6.75)
- added R1: 2.2k, Resistor_SMD:R_0402_1005Metric, F.Cu at (-28.8, 3.25)
- added R10: 0R, Resistor_SMD:R_0402_1005Metric, F.Cu at (-28.2, 14.8)
- added R100: 10k, Resistor_SMD:R_0402_1005Metric, F.Cu at (-21.2, -9.00)
- added R101: 10k, Resistor_SMD:R_0402_1005Metric, F.Cu at (-19.2, -6.75)
- added R11: 0R, Resistor_SMD:R_0402_1005Metric, F.Cu at (-27.2, 14.8)
- added R12: 100R, Resistor_SMD:R_0402_1005Metric, F.Cu at (-24.8, 14.5)
- added R13: 100R, Resistor_SMD:R_0402_1005Metric, F.Cu at (-24.8, 13.5)
- added R14: 100R, Resistor_SMD:R_0402_1005Metric, F.Cu at (-24.8, 12.5)
- added R17: 0R, Resistor_SMD:R_0402_1005Metric, F.Cu at (-24.8, 8.50)
- added R18: 0R, Resistor_SMD:R_0402_1005Metric, F.Cu at (-24.8, 7.50)
- added R2: 2.2k, Resistor_SMD:R_0402_1005Metric, F.Cu at (-28.8, 5.25)
- added R3: 100R, Resistor_SMD:R_0402_1005Metric, F.Cu at (-24.8, 15.5)
- added R4: 100R, Resistor_SMD:R_0402_1005Metric, F.Cu at (-27.2, 6.75)
- added R5: 100R, Resistor_SMD:R_0402_1005Metric, F.Cu at (-28.2, 6.74)
- added R6: 100R, Resistor_SMD:R_0402_1005Metric, F.Cu at (-24.8, 11.5)
- added R7: 100R, Resistor_SMD:R_0402_1005Metric, F.Cu at (-24.8, 10.5)
- added R8: 100R, Resistor_SMD:R_0402_1005Metric, F.Cu at (-24.8, 9.50)
- added R9: 10k, Resistor_SMD:R_0402_1005Metric, F.Cu at (-26.2, 6.75)
- added U100: STM32F042G4Ux, Package_DFN_QFN:QFN-28_4x4mm_P0.5mm, F.Cu at (-28.8, 10.8)
- J101: value Conn_01x03_Male -> JST_XH_S3B; footprint Connector_JST:JST_PH_B3B-PH-SM4-TB_1x03-1MP_P2.00mm_Vertical -> Connector_JST:JST_XH_S3B-XH-A_1x03_P2.50mm_Horizontal
- J102: value Conn_01x02_Male -> JST_XH_S4B; footprint Connector_JST:JST_PH_B2B-PH-SM4-TB_1x02-1MP_P2.00mm_Vertical -> Connector_JST:JST_XH_S4B-XH-A_1x04_P2.50mm_Horizontal
- J103: value Conn_01x02_Male -> USB_OTG; footprint Connector_JST:JST_PH_B2B-PH-SM4-TB_1x02-1MP_P2.00mm_Vertical -> Connector_USB:USB_Micro-B_Molex-105017-0001
- PCB100: value Board_Module -> 70x43
- moved J103 233.6 mm to (-28.0, 18.8), turned to 0 degrees
- moved J101 204.2 mm to (-20.0, 12.2), turned to 0 degrees
- moved R402 188.0 mm to (-11.5, -4.50), turned to 180 degrees
- moved R415 186.3 mm to (31.2, 7.25), turned to 0 degrees
- moved C410 183.9 mm to (31.8, 8.50), turned to 180 degrees
- moved PCB100 183.7 mm to (0.00, 0.00)
- moved J100 183.6 mm to (-33.2, 11.4)
- moved FB200 183.5 mm to (-27.2, 2.75), turned to 270 degrees
- moved J102 182.9 mm to (30.8, 3.75), turned to 90 degrees
- moved C407 182.3 mm to (16.2, 8.75), turned to 90 degrees
- moved C307 182.1 mm to (16.2, -16.2), turned to 90 degrees
- moved C419 181.9 mm to (24.2, 20.0), turned to 0 degrees
- moved C319 181.7 mm to (24.2, -5.00), turned to 0 degrees
- moved C420 181.0 mm to (24.8, 18.5), turned to 0 degrees
- moved C200 181.0 mm to (-24.8, 5.25)
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Connections:
- net /SPI_MISO renamed /RESERVED
- C201 pad 2: GNDA -> GND
- C203 pad 2: GNDA -> GND
- C204 pad 2: GNDA -> GND
- C205 pad 2: GNDA -> GND
- C206 pad 2: GNDA -> GND
- C207 pad 2: GNDA -> GND
- C300 pad 1: GNDA -> GND
- C301 pad 2: GNDA -> GND
- C306 pad 1: GNDA -> GND
- C307 pad 2: GNDA -> GND
- C308 pad 1: GNDA -> GND
- C310 pad 1: GNDA -> GND
- C311 pad 1: GNDA -> GND
- C312 pad 1: GNDA -> GND
- C313 pad 2: GNDA -> GND
- C314 pad 2: GNDA -> GND
- C315 pad 1: GNDA -> GND
- C316 pad 1: GNDA -> GND
- C317 pad 2: GNDA -> GND
- C318 pad 2: GNDA -> GND
- C319 pad 1: GNDA -> GND
- C320 pad 1: GNDA -> GND
- C321 pad 2: GNDA -> GND
- C322 pad 2: GNDA -> GND
- C400 pad 1: GNDA -> GND
- C401 pad 2: GNDA -> GND
- C406 pad 1: GNDA -> GND
- C407 pad 2: GNDA -> GND
- C408 pad 1: GNDA -> GND
- C410 pad 1: GNDA -> GND
- C411 pad 1: GNDA -> GND
- C412 pad 1: GNDA -> GND
- C413 pad 2: GNDA -> GND
- C414 pad 2: GNDA -> GND
- C415 pad 1: GNDA -> GND
- C416 pad 1: GNDA -> GND
- C417 pad 2: GNDA -> GND
- C418 pad 2: GNDA -> GND
- C419 pad 1: GNDA -> GND
- C420 pad 1: GNDA -> GND
- C421 pad 2: GNDA -> GND
- C422 pad 2: GNDA -> GND
- J100 pad 1: /I2S_MCLK -> +3V3
- J100 pad 10: Net-(J100-Pad10) -> GND
- J100 pad 12: /SPI_CS -> GND
- J100 pad 13: /SPI_SCK -> /I2S_SD0
- J100 pad 14: /SPI_MOSI -> GND
- J100 pad 15: /SHDN -> /I2S_LRCLK
- J100 pad 16: /MUTE -> GND
- J100 pad 17: GND -> /I2S_BCLK
- J100 pad 19: +3V3 -> /I2S_MCLK
- J100 pad 2: GND -> +5V
- J100 pad 20: +5V -> GND
- J100 pad 3: /I2S_LRCLK -> /nMUTE
- J100 pad 5: /I2S_BCLK -> /ENABLE
- J100 pad 7: /I2S_SDI -> /I2C_SDA
- J100 pad 9: Net-(J100-Pad9) -> /I2C_SCL
- J101 pad 2: GNDA -> GND
- J102 pad 1: /Left Buffer/Out -> /Right Buffer/Out
- J102 pad 2: GNDA -> GND
- J103 pad 1: /Right Buffer/Out -> Net-(J103-Pad1)
- J103 pad 2: GNDA -> /USB_DM
- PCB100 pad 3: GNDA -> GND
- PCB100 pad 4: GNDA -> GND
- R201 pad 2: GNDA -> GND
- R202 pad 2: GNDA -> GND
- R310 pad 2: GNDA -> GND
- R315 pad 2: GNDA -> GND
- R410 pad 2: GNDA -> GND
- R415 pad 2: GNDA -> GND
- U200 pad 10: GNDA -> GND
- U200 pad 19: GNDA -> GND
- U200 pad 23: /SHDN -> /ENABLE
- U200 pad 4: /I2S_SDI -> /I2S_SD0
Routing:
- net +15V: track 25.6 -> 164.5 mm, vias 2 -> 8
- net -15V: track 21.4 -> 149.1 mm, vias 0 -> 4
- net GNDA: track 56.4 -> 0.00 mm, vias 52 -> 1
- net /nMUTE: track 0.00 -> 41.8 mm
- net /ENABLE: track 0.00 -> 40.4 mm
- net +3V3: track 0.00 -> 36.0 mm, vias 0 -> 3
- net GND: track 1.58 -> 34.6 mm, vias 2 -> 728
- net Net-(R302-Pad1): track 0.00 -> 27.3 mm, vias 0 -> 2
- net /I2S_SD0: track 0.00 -> 26.0 mm
- net Net-(C305-Pad2): track 3.70 -> 22.0 mm
- net Net-(C405-Pad2): track 3.70 -> 21.8 mm
- net Net-(R402-Pad1): track 18.4 -> 34.4 mm
- net /I2S_BCLK: track 10.9 -> 26.0 mm
- net /I2S_LRCLK: track 11.1 -> 26.0 mm
- net /I2C_SCL: track 0.00 -> 12.0 mm
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- added copper zone on F.Cu, net GND
- removed copper zone on B.Cu, net GNDA
Other:
- board text added: "Farving Acoustics FA-DAC 1000005-2.0.0"
